File: schematic/v0.2/magspoof.kicad_pcb (KiCad board)
At the start: 2 copper layers, 29.2 x 39.4 mm, 24 parts, among them IC1 STM32F042G6U6, IC3 DRV8835DSSR, P1 USB_A, P2 Expansion Port, P3 Ext Clock, P4 Program Port, U1 MCP73831-2-OT

Commit message: PCB ordered
Routing:
- net SWDIO: track 25.1 -> 17.8 mm
- net GND: track 49.6 -> 47.5 mm, vias 8 -> 6
- net RESET: track 12.2 -> 11.2 mm, vias 0 -> 1
Changed lines of the file:
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@@
     (thickness 1.6)
     (drawings 20)
-    (tracks 311)
+    (tracks 295)
     (zones 0)
     (modules 24)
@@
   (segment (start 154.873 105.4065) (end 154.1585 105.4065) (width 0.254) (layer F.Cu) (net 1))
   (segment (start 154.1585 105.4065) (end 153.6585 104.9065) (width 0.254) (layer F.Cu) (net 1))
-  (via (at 140.716 105.4735) (size 0.6858) (drill 0.3302) (layers F.Cu B.Cu) (net 2))
-  (via (at 140.716 107.5055) (size 0.6858) (drill 0.3302) (layers F.Cu B.Cu) (net 2))
-  (segment (start 140.716 105.4735) (end 140.716 107.5055) (width 0.254) (layer B.Cu) (net 2))
   (via (at 147.574 101.854) (size 0.6858) (drill 0.3302) (layers F.Cu B.Cu) (net 2))
   (via (at 143.891 101.854) (size 0.6858) (drill 0.3302) (layers F.Cu B.Cu) (net 2))
@@
   (segment (start 155.3845 106.2355) (end 155.321 106.2355) (width 0.254) (layer B.Cu) (net 10))
   (segment (start 155.321 106.2355) (end 151.5745 106.2355) (width 0.254) (layer B.Cu) (net 10))
-  (segment (start 147.28825 106.52125) (end 147.2565 106.553) (width 0.254) (layer F.Cu) (net 11))
-  (segment (start 147.2565 106.553) (end 139.573 106.553) (width 0.254) (layer F.Cu) (net 11))
-  (segment (start 139.573 106.553) (end 138.43 105.41) (width 0.254) (layer F.Cu) (net 11))
-  (segment (start 149.4585 104.9065) (end 149.454 104.902) (width 0.254) (layer F.Cu) (net 11))
-  (segment (start 149.454 104.902) (end 148.844 104.902) (width 0.254) (layer F.Cu) (net 11))
-  (segment (start 148.844 104.902) (end 148.844 104.9655) (width 0.254) (layer F.Cu) (net 11))
-  (segment (start 148.844 104.9655) (end 147.28825 106.52125) (width 0.254) (layer F.Cu) (net 11))
+  (segment (start 149.4585 104.9065) (end 149.454 104.902) (width 0.254) (layer F.Cu) (net 11) (status C00000))
+  (segment (start 149.454 104.902) (end 148.082 104.902) (width 0.254) (layer F.Cu) (net 11) (status 400000))
+  (segment (start 148.082 104.902) (end 138.938 104.902) (width 0.254) (layer B.Cu) (net 11) (status 800000))
+  (via (at 148.082 104.902) (size 0.6858) (drill 0.3302) (layers F.Cu B.Cu) (net 11))
+  (segment (start 138.938 104.902) (end 138.43 105.41) (width 0.254) (layer B.Cu) (net 11) (status C00000))
   (segment (start 147.32 111.8) (end 147.959196 111.8) (width 0.254) (layer F.Cu) (net 13))
   (segment (start 148.919 105.9065) (end 149.4585 105.9065) (width 0.254) (layer F.Cu) (net 13))
@@
   (segment (start 152.93975 97.37725) (end 151.41575 95.85325) (width 0.254) (layer F.Cu) (net 22))
   (segment (start 151.41575 95.85325) (end 151.384 95.8215) (width 0.254) (layer F.Cu) (net 22))
-  (via (at 150.4315 106.045) (size 0.6858) (drill 0.3302) (layers F.Cu B.Cu) (net 23))
-  (segment (start 150.4315 106.045) (end 146.05 106.045) (width 0.254) (layer B.Cu) (net 23))
-  (segment (start 140.081 106.299) (end 138.43 107.95) (width 0.254) (layer B.Cu) (net 23))
-  (segment (start 140.081 102.5525) (end 140.081 106.299) (width 0.254) (layer B.Cu) (net 23))
-  (segment (start 140.5255 102.5525) (end 140.081 102.5525) (width 0.254) (layer B.Cu) (net 23))
-  (segment (start 141.351 102.5525) (end 140.5255 102.5525) (width 0.254) (layer B.Cu) (net 23))
-  (segment (start 142.24 102.5525) (end 141.351 102.5525) (width 0.254) (layer B.Cu) (net 23))
-  (segment (start 142.24 105.4735) (end 142.24 102.5525) (width 0.254) (layer B.Cu) (net 23))
-  (segment (start 145.542 105.4735) (end 142.24 105.4735) (width 0.254) (layer B.Cu) (net 23))
-  (segment (start 145.542 105.664) (end 145.542 105.4735) (width 0.254) (layer B.Cu) (net 23))
-  (segment (start 145.542 105.7275) (end 145.542 105.664) (width 0.254) (layer B.Cu) (net 23))
-  (segment (start 145.542 106.045) (end 145.542 105.7275) (width 0.254) (layer B.Cu) (net 23))
-  (segment (start 146.05 106.045) (end 145.542 106.045) (width 0.254) (layer B.Cu) (net 23))
-  (segment (start 151.765 103.4415) (end 151.7015 103.4415) (width 0.254) (layer F.Cu) (net 23))
-  (segment (start 151.7015 103.4415) (end 151.7015 103.5685) (width 0.254) (layer F.Cu) (net 23))
-  (segment (start 151.7015 103.5685) (end 151.257 104.013) (width 0.254) (layer F.Cu) (net 23))
-  (segment (start 151.765 103.4415) (end 153.6235 103.4415) (width 0.254) (layer F.Cu) (net 23))
-  (segment (start 151.3205 105.156) (end 150.4315 106.045) (width 0.254) (layer F.Cu) (net 23))
-  (segment (start 151.3205 104.0765) (end 151.3205 105.156) (width 0.254) (layer F.Cu) (net 23))
-  (segment (start 151.257 104.013) (end 151.3205 104.0765) (width 0.254) (layer F.Cu) (net 23))
-  (segment (start 153.6585 103.4065) (end 153.6235 103.4415) (width 0.254) (layer F.Cu) (net 23))
+  (segment (start 151.3205 104.013) (end 151.257 104.0765) (width 0.254) (layer F.Cu) (net 23))
+  (segment (start 151.9555 103.378) (end 151.3205 104.013) (width 0.254) (layer F.Cu) (net 23))
+  (segment (start 153.63 103.378) (end 151.9555 103.378) (width 0.254) (layer F.Cu) (net 23) (status 400000))
+  (segment (start 140.3985 105.9815) (end 138.43 107.95) (width 0.254) (layer B.Cu) (net 23) (status 800000))
+  (segment (start 150.4315 105.9815) (end 140.3985 105.9815) (width 0.254) (layer B.Cu) (net 23))
+  (via (at 150.4315 105.9815) (size 0.6858) (drill 0.3302) (layers F.Cu B.Cu) (net 23))
+  (segment (start 151.257 105.156) (end 150.4315 105.9815) (width 0.254) (layer F.Cu) (net 23))
+  (segment (start 151.257 104.0765) (end 151.257 105.156) (width 0.254) (layer F.Cu) (net 23))
+  (segment (start 153.6585 103.4065) (end 153.63 103.378) (width 0.254) (layer F.Cu) (net 23) (status C00000))
+  (segment (start 153.6585 103.4065) (end 153.6235 103.4415) (width 0.254) (layer F.Cu) (net 23) (status C00000))
   (segment (start 156.972 105.6005) (end 159.258 107.8865) (width 0.254) (layer B.Cu) (net 24))
   (segment (start 153.3125 102.5525) (end 153.9875 102.5525) (width 0.254) (layer F.Cu) (net 24))
